File: PCB/M.Seade Keypad.kicad_pcb (KiCad board)
At the start: 2 copper layers, 68.8 x 55.8 mm, 7 parts, among them J1 OLED_DISPLAY, SW1 Button, SW2 Button, SW3 Button, SW6 Button, SW8 Rotary Encoder, U1 XIAO-RP2040-DIP

Commit message: Add files via upload
Parts:
- SW1, SW2, SW3, SW6: value Button -> SW_Push
- SW8: value Rotary Encoder -> RotaryEncoder_Switch
Routing:
- net SCL: track 8.64 -> 28.9 mm
- net EC11SWB: track 82.7 -> 62.5 mm
- net GND: track 173.1 -> 167.5 mm
- net EC11B: track 37.6 -> 35.3 mm
- net EC11SWA: track 71.1 -> 69.6 mm
- net SW3: track 81.8 -> 82.9 mm
